File: hw/svetofor.sch (KiCad schematic (older format))
At the start: 61 parts

Commit message: HW PCB
Parts:
- removed D? (x9): LED_RGBA, LED_SMD:LED_SK6812MINI_PLCC4_3.5x3.5mm_P1.75mm, symbol Device:LED_RGBA
- removed R? (x27): R, Resistor_SMD:R_0603_1608Metric, symbol Device:R
- added C5: 100nF, Capacitor_SMD:C_0603_1608Metric, symbol Device:C
- added D1, D2, D3: LED_RGBA, LED_SMD:LED_SK6812MINI_PLCC4_3.5x3.5mm_P1.75mm, symbol Device:LED_RGBA
- added J10: SV1, Connector_PinHeader_2.54mm:PinHeader_1x04_P2.54mm_Vertical, symbol Connector_Generic:Conn_01x04
- added J11: SV2, Connector_PinHeader_2.54mm:PinHeader_1x04_P2.54mm_Vertical, symbol Connector_Generic:Conn_01x04
- added J2: I2C, Connector_PinHeader_2.54mm:PinHeader_1x03_P2.54mm_Vertical, symbol Connector_Generic:Conn_01x03
- added Q1, Q2, Q3, Q4, Q5, Q6: IRLML2060, Package_TO_SOT_SMD:SOT-23, symbol Transistor_FET:IRLML2060
- added R1, R2, R3, R4, R5, R6, R7, R8, R9: R, Resistor_SMD:R_0603_1608Metric, symbol Device:R
- D7: renamed from D?; footprint (none) -> LED_SMD:LED_0402_1005Metric
- J1: renamed from J?; value Conn_01x02_Female -> 5V; footprint (none) -> Connector_PinSocket_2.54mm:PinSocket_1x02_P2.54mm_Vertical
- J3: renamed from J?; footprint (none) -> Connector_PinHeader_2.54mm:PinHeader_2x05_P2.54mm_Vertical
- SW1: renamed from SW?; footprint (none) -> Button_Switch_SMD:SW_SPST_B3U-1000P-B
- Y1: renamed from Y?; footprint Crystal:Crystal_HC18-U_Vertical -> Crystal:Crystal_HC49-4H_Vertical
- gave numbers to parts that had none: 20
Connections:
- net GND: now also C5.2, J2.3 (Pin_3), Q1.2 (S), Q2.2 (S), Q3.2 (S), Q4.2 (S), Q5.2 (S), Q6.2 (S)
- net GREEN1: now also J10.4 (Pin_4), J11.4 (Pin_4), Q2.1 (G), Q5.1 (G); no longer R37.2
- net RED1: now also J10.2 (Pin_2), J11.2 (Pin_2), Q3.1 (G), Q6.1 (G); no longer R33.2
- net VCC: now also C5.1, D1.4 (A), D2.4 (A), D3.4 (A), J10.1 (Pin_1), J11.1 (Pin_1)
- net YELLOW1: now also J10.3 (Pin_3), J11.3 (Pin_3), Q1.1 (G), Q4.1 (G); no longer R30.2, R31.2
- net I2C_SDA: now reaches U2.27 (PC4)
- net I2C_SDA: now also J2.1 (Pin_1)
- net I2C_SCK: now reaches U2.28 (PC5)
- net I2C_SCK: now also J2.2 (Pin_2)
- new net: Q6.3 (D), R33.2
- new net: Q4.3 (D), R30.2, R31.2
- new net: Q5.3 (D), R37.2
- new net: Q2.3 (D), R8.2
- new net: Q1.3 (D), R4.2, R5.2
- new net: D1.1 (RK), R1.1
- new net: D1.2 (GK), R2.1
- new net: D1.3 (BK), R3.1
- new net: Q3.3 (D), R1.2
- new net: D2.1 (RK), R4.1
- new net: D2.2 (GK), R5.1
- new net: D2.3 (BK), R6.1
- new net: D3.1 (RK), R7.1
- new net: D3.2 (GK), R8.1
- new net: D3.3 (BK), R9.1
Other:
- moved on the sheet: D11, D12, D13, J3, R30, R31, R32, R33, R34, R35, R36, R37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
